Commit message: 完善检测抓取流程

File: mujoco/urdf/mujoco_ros2_control.xacro (robot description, xacro)
@@ -7,4 +7,6 @@
         <param name="mujoco_model">${mujoco_model_path}</param>
         <param name="headless">${headless}</param>
+        <param name="sim_speed_factor">1.0</param>
+        <param name="camera_publish_rate">10.0</param>
       </hardware>
       <joint name="shoulder_pan_joint">
@@ -50,4 +52,10 @@
         <state_interface name="effort"/>
       </joint>
+      <sensor name="gemini2_camera">
+        <param name="frame_name">gemini2_camera_frame</param>
+        <param name="info_topic">/env_0/gemini2/camera_info</param>
+        <param name="image_topic">/env_0/gemini2/rgb</param>
+        <param name="depth_topic">/env_0/gemini2/depth</param>
+      </sensor>
     </ros2_control>
   </xacro:macro>

File: mujoco/urdf/ur5e_mujoco.urdf.xacro (robot description, xacro)
@@ -28,5 +28,5 @@
     generate_ros2_control_tag="false"
     headless_mode="false"
-    initial_positions="${dict(shoulder_pan_joint=0.0,shoulder_lift_joint=-1.57,elbow_joint=0.0,wrist_1_joint=-1.57,wrist_2_joint=0.0,wrist_3_joint=0.0)}"
+    initial_positions="${dict(shoulder_pan_joint=0.0,shoulder_lift_joint=-1.57,elbow_joint=1.57,wrist_1_joint=0.0,wrist_2_joint=1.57,wrist_3_joint=0.0)}"
     robot_ip="0.0.0.0"
     >

File: src/moveit_config/srdf/ur_macro.srdf.xacro (robot description, xacro)
@@ -8,9 +8,9 @@
     </group>
     <group_state name="${prefix}home" group="${prefix}${name}_manipulator">
-      <joint name="${prefix}elbow_joint" value="0" />
+      <joint name="${prefix}elbow_joint" value="1.5707" />
       <joint name="${prefix}shoulder_lift_joint" value="-1.5707" />
       <joint name="${prefix}shoulder_pan_joint" value="0" />
       <joint name="${prefix}wrist_1_joint" value="0" />
-      <joint name="${prefix}wrist_2_joint" value="0" />
+      <joint name="${prefix}wrist_2_joint" value="1.5707" />
       <joint name="${prefix}wrist_3_joint" value="0" />
     </group_state>
